Commit message: 当たり判定を追加。一旦4軸に変更。

File: src/frontend/public/urdf/dummy_arm.urdf (robot description, URDF)
Before this commit: robot dummy_arm, 11 links, 10 joints
Links:
- removed link link5
- removed link link6
- link gripper_base: geometry visual box size=0.12 0.04 0.02
- link link4: geometry visual box size=0.08 0.08 0.06; visual sphere radius=0.06
Joints:
- removed joint joint5
- removed joint joint6
- joint gripper_base_joint: origin xyz=0 0.1 0 rpy=0 0 0 -> xyz=0 0.08 0 rpy=0 0 0; parent link6 -> link4
- joint joint1: axis 0 0 1 -> 0 1 0; origin xyz=0 0 0.05 rpy=0 0 0 -> xyz=0 0.05 0 rpy=0 0 0
- joint joint2: axis 0 1 0 -> 0 0 1; origin xyz=0 0 0.15 rpy=0 0 0 -> xyz=0 0.15 0 rpy=0 0 0
- joint joint3: axis 0 1 0 -> 0 0 1; limit lower=-3.14 upper=3.14 effort=10.0 velocity=1.0 -> lower=0.0 upper=3.14 effort=10.0 velocity=1.0; origin xyz=0 0 0.3 rpy=0 0 0 -> xyz=0 0.3 0 rpy=0 0 0
- joint joint4: axis 0 1 0 -> 0 0 1; origin xyz=0 0 0.25 rpy=0 0 0 -> xyz=0 0.25 0 rpy=0 0 0
- joint left_finger_joint: origin xyz=-0.05 0.02 0 rpy=0 0 0 -> xyz=-0.05 0.04 0 rpy=0 0 0
- joint right_finger_joint: origin xyz=0.05 0.02 0 rpy=0 0 0 -> xyz=0.05 0.04 0 rpy=0 0 0

Commit message: 6軸アームに変更

File: src/frontend/public/urdf/dummy_arm.urdf (robot description, URDF)
Before this commit: robot dummy_arm, 9 links, 8 joints
Links:
- added link link5; visual cylinder length=0.04 radius=0.03; visual sphere radius=0.05
- added link link6; visual box size=0.06 0.02 0.06; visual sphere radius=0.04
- link link4: geometry visual cylinder length=0.06 radius=0.04; visual sphere radius=0.06
Joints:
- added joint joint5: type revolute, parent link4, child link5, origin xyz=0 0.06 0 rpy=0 0 0, axis 1 0 0, limit lower=-3.14 upper=3.14 effort=10.0 velocity=1.0
- added joint joint6: type revolute, parent link5, child link6, origin xyz=0 0.04 0 rpy=0 0 0, axis 0 1 0, limit lower=-3.14 upper=3.14 effort=10.0 velocity=1.0
- joint gripper_base_joint: origin xyz=0 0.08 0 rpy=0 0 0 -> xyz=0 0.02 0 rpy=0 0 0; parent link4 -> link6

Commit message: 腕と手首の違いを分かりやすくした。操作パネルを変更した。

File: src/frontend/public/urdf/dummy_arm.urdf (robot description, URDF)
Before this commit: robot dummy_arm, 11 links, 10 joints
Links:
- link link3: geometry visual cylinder length=0.25 radius=0.03; visual sphere radius=0.07
- link link4: geometry visual cylinder length=0.06 radius=0.025; visual sphere radius=0.035
- link link5: geometry visual cylinder length=0.04 radius=0.02; visual sphere radius=0.03
- link link6: geometry visual box size=0.04 0.02 0.04; visual sphere radius=0.025

Commit message: オブジェクトを掴めるように調整

File: src/frontend/public/urdf/dummy_arm.urdf (robot description, URDF)
Before this commit: robot dummy_arm, 11 links, 10 joints
Links:
- link left_finger: geometry visual box size=0.01 0.06 0.08
- link right_finger: geometry visual box size=0.01 0.06 0.08

Commit message: アームの動きを調整

File: src/frontend/public/urdf/dummy_arm.urdf (robot description, URDF)
Before this commit: robot dummy_arm, 11 links, 10 joints
Links:
- added link floor; collision box size=4.0 0.1 4.0
Joints:
- added joint floor_joint: type fixed, parent base_link, child floor, origin xyz=0 0 0 rpy=0 0 0
- joint joint2: limit lower=-3.14 upper=3.14 effort=10.0 velocity=1.0 -> lower=-1.57 upper=1.57 effort=10.0 velocity=1.0

File: src/robot/urdf/dummy_arm.urdf (robot description, URDF)
Before this commit: robot dummy_arm, 11 links, 10 joints
Links:
- added link floor; collision box size=4.0 0.1 4.0
Joints:
- added joint floor_joint: type fixed, parent base_link, child floor, origin xyz=0 0 0 rpy=0 0 0
- joint joint2: limit lower=-3.14 upper=3.14 effort=10.0 velocity=1.0 -> lower=-1.57 upper=1.57 effort=10.0 velocity=1.0
